Commit message: updated

File: src/husarion_components_description/urdf/orbbec_astra.urdf.xacro (robot description, xacro)
@@ -42,5 +42,5 @@
         <origin xyz="0.0 0.0 0.0" rpy="${pi/2} 0.0 0.0" />
         <geometry>
-          <mesh filename="package://husarion_components_description/meshes/orbbec_astra.glb" />
+          <mesh filename="package://husarion_components_description/meshes/orbbec_astra.dae" />
         </geometry>
       </visual>

File: src/husarion_components_description/urdf/slamtec_rplidar.urdf.xacro (robot description, xacro)
@@ -38,5 +38,5 @@
       <xacro:property name="dist_res" value="0.01" />
       <xacro:property name="std_dev" value="0.015" />
-      <xacro:property name="mesh" value="s3.glb" />
+      <xacro:property name="mesh" value="s3.dae" />
       <xacro:property name="collision">
         <origin xyz="0.0 0.0 ${0.0413/2.0}" rpy="0.0 0.0 0.0" />
@@ -63,5 +63,5 @@
       <xacro:property name="dist_res" value="0.013" />
       <xacro:property name="std_dev" value="0.015" />
-      <xacro:property name="mesh" value="s2.glb" />
+      <xacro:property name="mesh" value="s2.dae" />
       <xacro:property name="collision">
         <origin xyz="0.0 0.0 ${0.038857/2.0}" rpy="0.0 0.0 0.0" />
@@ -88,5 +88,5 @@
       <xacro:property name="dist_res" value="0.03" />
       <xacro:property name="std_dev" value="0.025" />
-      <xacro:property name="mesh" value="s1.glb" />
+      <xacro:property name="mesh" value="s1.dae" />
       <xacro:property name="collision">
         <origin xyz="0.0 0.0 0.025" rpy="0.0 0.0 0.0" />
@@ -113,5 +113,5 @@
       <xacro:property name="dist_res" value="0.015" />
       <xacro:property name="std_dev" value="0.02" />
-      <xacro:property name="mesh" value="c1.glb" />
+      <xacro:property name="mesh" value="c1.dae" />
       <xacro:property name="collision">
         <origin xyz="0.0 0.0 ${0.0413/2.0}" rpy="0.0 0.0 0.0" />
@@ -139,5 +139,5 @@
       <xacro:property name="dist_res" value="0.03" />
       <xacro:property name="std_dev" value="0.05" />
-      <xacro:property name="mesh" value="a3.glb" />
+      <xacro:property name="mesh" value="a3.dae" />
       <xacro:property name="collision">
         <origin xyz="0.0 0.0 ${0.041/2.0}" rpy="0.0 0.0 0.0" />
@@ -164,5 +164,5 @@
       <xacro:property name="dist_res" value="0.03" />
       <xacro:property name="std_dev" value="0.05" />
-      <xacro:property name="mesh" value="a2.glb" />
+      <xacro:property name="mesh" value="a2.dae" />
       <xacro:property name="collision">
         <origin xyz="0.0 0.0 ${0.041/2.0}" rpy="0.0 0.0 0.0" />
@@ -188,5 +188,5 @@
       <xacro:property name="dist_res" value="0.03" />
       <xacro:property name="std_dev" value="0.05" />
-      <xacro:property name="mesh" value="a2.glb" />
+      <xacro:property name="mesh" value="a2.dae" />
       <xacro:property name="collision">
         <origin xyz="0.0 0.0 ${0.041/2.0}" rpy="0.0 0.0 0.0" />
@@ -212,5 +212,5 @@
       <xacro:property name="dist_res" value="0.03" />
       <xacro:property name="std_dev" value="0.05" />
-      <xacro:property name="mesh" value="a2.glb" />
+      <xacro:property name="mesh" value="a2.dae" />
       <xacro:property name="collision">
         <origin xyz="0.0 0.0 ${0.041/2.0}" rpy="0.0 0.0 0.0" />
@@ -265,8 +265,8 @@
           <scan>
             <horizontal>
-              <samples>${samples}</samples>
+              <samples>${int(samples * 8/9)}</samples>
               <resolution>1</resolution>
-              <min_angle>-${pi}</min_angle>
-              <max_angle>${pi}</max_angle>
+              <min_angle>${pi/9}</min_angle>
+              <max_angle>${17*pi/9}</max_angle>
             </horizontal>
           </scan>

File: src/husarion_components_description/urdf/velodyne_puck.urdf.xacro (robot description, xacro)
@@ -39,5 +39,5 @@
         <origin xyz="0.0 0.0 0.0" rpy="${pi/2} 0.0 0.0" />
         <geometry>
-          <mesh filename="package://husarion_components_description/meshes/velodyne_puck.glb" />
+          <mesh filename="package://husarion_components_description/meshes/velodyne_puck.dae" />
         </geometry>
       </visual>

File: src/rosbot_description/urdf/rosbot_xl.urdf.xacro (robot description, xacro)
@@ -4,4 +4,5 @@
   <xacro:arg name="configuration" default="basic" />
   <xacro:arg name="controller_config" default="" />
+  <xacro:arg name="include_antenna" default="False" />
   <xacro:arg name="include_camera_mount" default="False" />
   <xacro:arg name="manipulator_serial_port" default="/dev/ttyUSB0" />
@@ -17,4 +18,5 @@
   <xacro:husarion.rosbot_xl
     controller_config="$(arg controller_config)"
+    include_antenna="$(arg include_antenna)"
     include_camera_mount="$(arg include_camera_mount)"
     mecanum="$(arg mecanum)"

File: src/rosbot_description/urdf/rosbot_xl/rosbot_xl_macro.urdf.xacro (robot description, xacro)
@@ -3,4 +3,5 @@
   <xacro:macro name="rosbot_xl"
     params="controller_config
+            include_antenna:=False
             include_camera_mount
             mecanum
@@ -19,5 +20,7 @@
     <!-- BODY -->
     <xacro:body.body wheel_radius="${wheel_radius}" />
-    <xacro:antenna.antenna parent_link="cover_link" xyz="-0.155 -0.055 -0.02" rpy="-0.4 0.0 0.0" antenna_angle="0.3" />
+    <xacro:if value="${include_antenna}">
+      <xacro:antenna.antenna parent_link="cover_link" xyz="-0.155 -0.055 -0.02" rpy="-0.4 0.0 0.0" antenna_angle="0.3" />
+    </xacro:if>
     <xacro:if value="${include_camera_mount}">
       <xacro:camera_mount.camera_mount parent_link="cover_link" xyz="-0.1 0.0 0.0" />
